File: hardware/Roomba_Lattepanda_seial_circuit/Schematics-2.brd (EAGLE design)
At the start: 32.7 x 25.4 mm, 14 parts

Commit message: update hardware
Parts:
- removed JP10, JP9: (no value), adafruit:1X03-CLEANBIG
- removed JP11, JP12: (no value), adafruit:1X01
- added GND, PWR, RX, SERVO_P, SERVO_R, TX: (no value), adafruit:1X01-CLEANBIG
- added NEOP, SERVO_P_PINS, SERVO_R_PINS: (no value), adafruit:1X03-CLEANBIG
- added SOFTS: (no value), con-lstb:MA04-1
- added U$1: 2.1MMJACKTHM, adafruit:PJ-102A
- JP1, JP7: value (none) -> NEO_D
- JP3: value (none) -> DBG
- moved JP8 29.2 mm to (8.57, 38.4)
- moved JP3 22.9 mm to (2.54, 27.9)
- moved JP2 20.3 mm to (8.57, 25.4)
- moved JP7 18.2 mm to (8.57, 27.9)
- moved JP5 13.2 mm to (8.57, 15.2)
- moved JP6 12.3 mm to (14.6, 20.0)
- moved R1 10.2 mm to (26.7, 30.5)
- moved DEBUG_S 10.2 mm to (27.3, 23.2)
- moved JP1 7.62 mm to (5.08, 25.4)
- moved JP4 2.56 mm to (10.2, 20.0)
Connections:
- removed net N$6: DEBUG_S.2, JP8.1, R1.1
- removed net N$7: JP2.1, JP9.2
- new net N$10: JP7.1, JP8.1, SERVO_R.1, SERVO_R_PINS.1
- new net N$12: SERVO_P.1, SERVO_P_PINS.1
- new net N$9: SERVO_P_PINS.2, SERVO_R_PINS.2, U$1.TIP
- net N$1: now also RX.1, SOFTS.2; no longer JP10.1, JP11.1
- net N$2: now also JP2.1, JP5.1, NEOP.2; no longer JP4.1
- net N$3: now also SOFTS.3, TX.1; no longer JP10.2, JP12.1
- net N$4: now also GND.1, NEOP.1, SERVO_P_PINS.3, SERVO_R_PINS.3, SOFTS.4, U$1.RING; no longer JP10.3, JP3.1, JP9.1
- net N$5: now also NEOP.3, PWR.1; no longer JP5.1, JP9.3
- net N$8: now also DEBUG_S.2, JP3.1, JP4.1, R1.1; no longer JP7.1
Routing:
- net N$4: track 37.3 -> 112.4 mm
- net N$10: track 0.00 -> 63.5 mm
- net N$9: track 0.00 -> 55.6 mm
- net N$12: track 0.00 -> 38.8 mm
- net N$6: track 29.2 -> 0.00 mm
- net N$8: track 14.2 -> 42.2 mm
- net N$3: track 0.00 -> 15.2 mm
- net N$1: track 0.00 -> 15.2 mm
- net N$7: track 8.89 -> 0.00 mm
- net N$2: track 3.81 -> 12.7 mm
Other:
- board size 32.7 x 25.4 mm -> 48.6 x 43.5 mm
